File: KiCAD/FDC.kicad_pcb (KiCad board)
At the start: 2 copper layers, 72.6 x 65.5 mm, 24 parts, among them J2 Conn_02x20_Odd_Even, J3 SD_Card, Q1 SSM3K324RLFCT-ND, Q2 SSM3K324RLFCT-ND, U1 SN74LVCC4245ADWR, U2 Pico, U3 SN74LVCC4245ADWR, U4 SN74LVCC4245ADWR, U5 SN74LVCC4245ADWR

Commit message: Update to the KiCAD folder
Parts:
- U2: footprint PiPico:RPi_Pico_SMD_TH -> MCU_RaspberryPi_and_Boards:RPi_Pico_SMD_TH
