File: KiCAD/FDC.kicad_sch (KiCad schematic)
At the start: 24 parts, among them J2 Conn_02x20_Odd_Even, J3 SD_Card, Q1 SSM3K324RLFCT-ND, Q2 SSM3K324RLFCT-ND, U1 SN74LVCC4245ADWR, U2 Pico, U3 SN74LVCC4245ADWR, U4 SN74LVCC4245ADWR, U5 SN74LVCC4245ADWR

Commit message: Update to the KiCAD folder
Parts:
- D1: Cost 0.72 -> 0.70
- D2: Cost (none) -> .28; Digikey 1727-3879-1-ND -> (none)
- J2: Cost (none) -> 3.69
- J3: Cost 4.30 -> 2.13
- Q1, Q2: Cost (none) -> .37
- U1, U3, U4, U5: Cost 1.82 -> 1.83
- U2: footprint PiPico:RPi_Pico_SMD_TH -> MCU_RaspberryPi_and_Boards:RPi_Pico_SMD_TH
